File: ATMega Dev Board.kicad_pcb (KiCad board)
At the start: 4 copper layers, 84 x 38.1 mm, 39 parts, among them J1 Conn_01x09, J2 Conn_01x04, J3 Conn_01x09, J4 SPI header, J5 USB-C_31-M-12, Q1 S8050, SW1 SW_SPST, SW2 SW_SPST, U1 ATmega32A-A, U2 CH340C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

Commit message: Added power OR-ing
Parts:
- added Q2: 2N7002, Package_TO_SOT_SMD:SOT-23, F.Cu at (147.2, 77.9)
- added Q3: HL6042, PCM_JLCPCB:Q_SOT-23, F.Cu at (143.2, 80.7)
- added Q4: HL6042, PCM_JLCPCB:Q_SOT-23, F.Cu at (139.2, 80.7)
- added R8: 330k, Resistor_SMD:R_0603_1608Metric, F.Cu at (139.7, 77.9)
- added R9: 330k, Resistor_SMD:R_0603_1608Metric, F.Cu at (143.2, 77.9)
- moved J2 1.85 mm to (126.6, 76.4)
- moved C9 0.18 mm to (123.5, 79.4)
Connections:
- C13 pad 2: VCC -> VBUS
- C15 pad 1: VCC -> VBUS
- D5 pad 5: VCC -> VSPI
- F1 pad 1: VCC -> VBUS
- J4 pad 2: VCC -> VSPI
- R11 pad 1: VCC -> VBUS
- U2 pad 16: VCC -> VBUS
Routing:
- net VSPI: track 0.00 -> 85.5 mm
- net VCC: track 198.3 -> 129.9 mm
- net VBUS: track 0.00 -> 47.2 mm
- net Net-(Q2-D): track 0.00 -> 4.26 mm
- net GND: track 51.3 -> 53.9 mm, vias 25 -> 27
- net /PA7: track 15.4 -> 14.6 mm
- net /PA4: track 10.1 -> 10.8 mm
- net /PA5: track 11.6 -> 12.3 mm
