File: ATMega Dev Board.kicad_sch (KiCad schematic)
At the start: 39 parts, among them J1 Conn_01x09, J2 Conn_01x04, J3 Conn_01x09, J4 SPI header, J5 USB-C_31-M-12, Q1 S8050, SW1 SW_SPST, SW2 SW_SPST, U1 ATmega32A-A, U2 CH340C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

Commit message: Added power OR-ing
Parts:
- added Q2: 2N7002, Package_TO_SOT_SMD:SOT-23, symbol Transistor_FET:2N7002
- added Q3, Q4: HL6042, PCM_JLCPCB:Q_SOT-23, symbol PCM_JLCPCB-Transistors:PMOS,HL6042
- added R8, R9: 330k, Resistor_SMD:R_0603_1608Metric, symbol Device:R_Small
Connections:
- net GND: now also Q2.2 (S), R8.1
- net VCC: now also Q3.2 (S), Q4.2 (S), R9.1; no longer C13.2, C15.1, D5.5 (VP), F1.1, J4.2 (VCC), R11.1, U2.16 (VCC)
- new net: Q2.3 (D), Q3.1 (G), R9.2
- new net VBUS: C13.2, C15.1, F1.1, Q2.1 (G), Q3.3 (D), Q4.1 (G), R11.1, R8.2, U2.16 (VCC)
- new net VSPI: D5.5 (VP), J4.2 (VCC), Q4.3 (D)
Other:
- note added: "D"
- note added: "G"
- note added: "S"
- moved on the sheet: D3, LS1, Q1, R4, SW1, SW2
